File: Keyboards/Waffle/kicad/Pancake_v8.kicad_pcb (KiCad board)
At the start: 4 copper layers, 115.5 x 76.2 mm, 91 parts, among them J1 HRO_TYPE-C-31-M-14, J2 TC2030_SWD, J3 Battery, Q1 2N7002, SW1 SW_Push_45deg, SW10 SW_Push_45deg, SW11 SW_Push_45deg, SW12 SW_Push_45deg, SW13 SW_Push_45deg, SW14 SW_Push_45deg, SW15 SW_Push_45deg, SW16 SW_Push_45deg, SW17 SW_Push_45deg, SW18 SW_Push_45deg, SW19 SW_Push_45deg, SW2 SW_Push_45deg, SW20 SW_Push_45deg, SW21 SW_Push_45deg, SW22 SW_Push_45deg, SW23 SW_Push_45deg, SW24 SW_Push_45deg, SW25 SW_Push_45deg, SW26 SW_Push_45deg, SW27 RST, SW28 PWR, SW3 SW_Push_45deg, SW4 SW_Push_45deg, SW5 SW_Push_45deg, SW6 SW_Push_45deg, SW7 SW_Push_45deg, SW8 SW_Push_45deg, SW9 SW_Push_45deg, U1 SRV05-4, U2 BQ24075, U3 nRF52840_E73-2G4M08S1C, Y1 32.768 KHz

Commit message: Update waffle proto
Parts:
- added G***: LOGO, MyFiles:pancake3, F.Cu at (92.1, 90.4)
- R7, R9: value 1k5 -> 10k
- SW1, SW10, SW11, SW12, SW13, SW14, SW15, SW16, SW17, SW18, SW19, SW2, SW20, SW21, SW22, SW23, SW24, SW25, SW26, SW3, SW4, SW5, SW6, SW7, SW8, SW9: moved to F.Cu
- moved D3 19.1 mm to (72.4, 60.6)
- moved D4 17.9 mm to (91.5, 60.0)
- moved D2 17.9 mm to (54.6, 60.6)
- moved D8 16.7 mm to (54.6, 79.7)
- moved D12 13.0 mm to (134.5, 77.7), turned to 45 degrees
- moved D5 1.19 mm to (110.5, 60.6)
- moved D1 1.19 mm to (52.2, 60.6)
- moved D7 1.19 mm to (52.2, 79.7)
- turned D18 to -45 degrees
- turned SW1 to 0 degrees
- turned SW10 to 0 degrees
- turned SW11 to 0 degrees
- turned SW12 to -90 degrees
- turned SW13 to 180 degrees
- turned SW14 to 180 degrees
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Connections:
- U3 pad 41: r1 -> r0
- U3 pad 43: r0 -> r1
- U3 pad 9: unconnected-(U3-P0.31/AIN7-Pad9) -> c1
Routing:
- net c1: track 81.2 -> 141.6 mm, vias 0 -> 2
- net r1: track 121.4 -> 103.7 mm
- net Net-(D23-A): track 24.1 -> 7.16 mm
- net Net-(D22-A): track 6.26 -> 19.1 mm
- net Net-(D21-A): track 6.22 -> 17.9 mm
- net Net-(D14-A): track 14.1 -> 5.32 mm
- net Net-(D24-A): track 29.3 -> 20.8 mm
- net Net-(D9-A): track 14.2 -> 5.80 mm
- net Net-(D11-A): track 14.6 -> 6.40 mm
- net Net-(D13-A): track 15.2 -> 7.18 mm
- net Net-(D15-A): track 6.01 -> 13.6 mm
- net Net-(D17-A): track 5.95 -> 13.5 mm
- net Net-(D6-A): track 15.1 -> 7.59 mm
- net Net-(D20-A): track 6.22 -> 13.4 mm
- net Net-(D10-A): track 5.14 -> 12.2 mm
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Other:
- outline, holes or cut-outs redrawn
- copper layers 4 -> 2
